Commit message: 更新readme

File: resources/robots/YQZ-000/urdf/YQZ-000.urdf (robot description, URDF)
Before this commit: robot YQZ-000, 17 links, 16 joints
Links:
- link FL_calf_Link: geometry collision box size=0.035 0.030 0.28; visual mesh filename=../meshes/FL_calf_Link.STL
- link FL_foot_Link: geometry collision cylinder length=0.05 radius=0.106; visual mesh filename=../meshes/FL_foot_Link.STL
- link FL_hip_Link: geometry collision box size=0.10 0.060 0.08; visual mesh filename=../meshes/FL_hip_Link.STL
- link FL_thigh_Link: geometry collision box size=0.055 0.040 0.30; visual mesh filename=../meshes/FL_thigh_Link.STL
- link FR_calf_Link: geometry collision box size=0.035 0.030 0.28; visual mesh filename=../meshes/FR_calf_Link.STL
- link FR_foot_Link: geometry collision cylinder length=0.05 radius=0.106; visual mesh filename=../meshes/FR_foot_Link.STL
- link FR_hip_Link: geometry collision box size=0.10 0.060 0.08; visual mesh filename=../meshes/FR_hip_Link.STL
- link FR_thigh_Link: geometry collision box size=0.055 0.040 0.30; visual mesh filename=../meshes/FR_thigh_Link.STL
- link RL_calf_Link: geometry collision box size=0.035 0.030 0.28; visual mesh filename=../meshes/RL_calf_Link.STL
- link RL_foot_Link: geometry collision cylinder length=0.05 radius=0.106; visual mesh filename=../meshes/RL_foot_Link.STL
- link RL_hip_Link: geometry collision box size=0.10 0.060 0.08; visual mesh filename=../meshes/RL_hip_Link.STL
- link RL_thigh_Link: geometry collision box size=0.055 0.040 0.30; visual mesh filename=../meshes/RL_thigh_Link.STL
- link RR_calf_Link: geometry collision box size=0.035 0.030 0.28; visual mesh filename=../meshes/RR_calf_Link.STL
- link RR_foot_Link: geometry collision cylinder length=0.05 radius=0.106; visual mesh filename=../meshes/RR_foot_Link.STL
- link RR_hip_Link: geometry collision box size=0.10 0.060 0.08; visual mesh filename=../meshes/RR_hip_Link.STL
- link RR_thigh_Link: geometry collision box size=0.055 0.040 0.30; visual mesh filename=../meshes/RR_thigh_Link.STL
- link base_link: geometry collision box size=0.58 0.20 0.12; visual mesh filename=../meshes/base_link.STL
Joints:
- joint FL_calf_joint: limit lower=0 upper=3.9461894387591787 effort=1 velocity=1 -> lower=0 upper=3.9461894387591787 effort=120 velocity=30
- joint FL_foot_joint: limit (none) -> lower=-9999 upper=9999 effort=17 velocity=50; type continuous -> revolute
- joint FL_hip_joint: limit lower=-0.8203047484373349 upper=0.5585053606381855 effort=0 velocity=0 -> lower=-0.8203047484373349 upper=0.5585053606381855 effort=60 velocity=30
- joint FL_thigh_joint: limit lower=-2.357939819444339 upper=0.8691739674931761 effort=1 velocity=1 -> lower=-2.357939819444339 upper=0.8691739674931761 effort=60 velocity=30
- joint FR_calf_joint: limit lower=-3.9461894387591787 upper=0 effort=1 velocity=1 -> lower=-3.9461894387591787 upper=0 effort=120 velocity=30
- joint FR_foot_joint: limit (none) -> lower=-9999 upper=9999 effort=17 velocity=50; type continuous -> revolute
- joint FR_hip_joint: limit lower=-0.5585053606381855 upper=0.8203047484373349 effort=1 velocity=1 -> lower=-0.5585053606381855 upper=0.8203047484373349 effort=60 velocity=30
- joint FR_thigh_joint: limit lower=-0.8691739674931761 upper=2.357939819444339 effort=0 velocity=0 -> lower=-0.8691739674931761 upper=2.357939819444339 effort=60 velocity=30
- joint RL_calf_joint: limit lower=-3.9461894387591787 upper=0 effort=1 velocity=1 -> lower=-3.9461894387591787 upper=0 effort=120 velocity=30
- joint RL_foot_joint: limit (none) -> lower=-9999 upper=9999 effort=17 velocity=50; type continuous -> revolute
- joint RL_hip_joint: limit lower=-0.5585053606381855 upper=0.8203047484373349 effort=1 velocity=1 -> lower=-0.5585053606381855 upper=0.8203047484373349 effort=60 velocity=30
- joint RL_thigh_joint: limit lower=-0.8691739674931761 upper=2.357939819444339 effort=0 velocity=0 -> lower=-0.8691739674931761 upper=2.357939819444339 effort=60 velocity=30
- joint RR_calf_joint: limit lower=0 upper=3.9461894387591787 effort=1 velocity=1 -> lower=0 upper=3.9461894387591787 effort=120 velocity=30
- joint RR_foot_joint: limit (none) -> lower=-9999 upper=9999 effort=17 velocity=50; type continuous -> revolute
- joint RR_hip_joint: limit lower=-0.8203047484373349 upper=0.5585053606381855 effort=0 velocity=0 -> lower=-0.8203047484373349 upper=0.5585053606381855 effort=60 velocity=30
- joint RR_thigh_joint: limit lower=-2.357939819444339 upper=0.8691739674931761 effort=1 velocity=1 -> lower=-2.357939819444339 upper=0.8691739674931761 effort=60 velocity=30
